File: hardware/sad/sad.kicad_sch (KiCad schematic)
At the start: 30 parts, among them IC1 LP5012RUKR, U1 ATtiny1616-M

Commit message: charger
Parts:
- added C4, C5: 4.7uF, Package_TO_SOT_SMD:SOT-23-5, symbol Device:C
- added J1: USB_C_Receptacle_USB2.0_16P, symbol Connector:USB_C_Receptacle_USB2.0_16P
- added R3: 6.8k, Package_TO_SOT_SMD:SOT-23-5, symbol Device:R
- added R4: 4.7k, Package_TO_SOT_SMD:SOT-23-5, symbol Device:R
- added R5: 1M, Package_TO_SOT_SMD:SOT-23-5, symbol Device:R
- added U2: MCP73831-2-OT, Package_TO_SOT_SMD:SOT-23-5, symbol Battery_Management:MCP73831-2-OT
Connections:
- net GND: now also C4.1, C5.2, R3.2, R5.1, U2.2 (V_{SS})
- net VBAT: now also C5.1, U2.3 (V_{BAT})
- new net: R4.1, U2.1 (STAT)
- new net: R3.1, U2.5 (PROG)
- new net: J1.A1 (GND), J1.A12 (GND), J1.B1 (GND), J1.B12 (GND)
- new net: J1.A4 (VBUS), J1.A9 (VBUS), J1.B4 (VBUS), J1.B9 (VBUS)
- new net STAT: R4.2, R5.2
- new net VBUS: C4.2, U2.4 (V_{DD})
Other:
- note added: "Check for protection on the cell"
- moved on the sheet: BT1, C1, C2, C3, IC1, JP1, JP10, JP2, JP3, JP4, JP5, JP6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

Commit message: init sch finished
Parts:
- added C6, C7: 10nF, Package_TO_SOT_SMD:SOT-23-5, symbol Device:C
- added C8: 1uF, Package_SO:SOIC-8_3.9x4.9mm_P1.27mm, symbol Device:C
- added D1: 5V, Package_DFN_QFN:QFN-16-1EP_4x4mm_P0.65mm_EP2.1x2.1mm_ThermalVias, symbol Device:D_TVS
- added R10, R11: 4.7k, Package_TO_SOT_SMD:SOT-23-5, symbol Device:R
- added R12, R8, R9: 1k, Package_TO_SOT_SMD:SOT-23-5, symbol Device:R
- added R6, R7: 5.1k, Package_TO_SOT_SMD:SOT-23-5, symbol Device:R
- added SW1, SW2: SW_Push, Button_Switch_SMD:Nidec_Copal_CAS-120A, symbol Switch:SW_Push
- added TP12: UDPI, Relay_THT:Relay_DPDT_Schrack-RT2-FormC_RM5mm, symbol Connector:TestPoint
- added TP13: DBG_TX, Relay_THT:Relay_DPDT_Schrack-RT2-FormC_RM5mm, symbol Connector:TestPoint
- added TP14: GND, Relay_THT:Relay_DPDT_Schrack-RT2-FormC_RM5mm, symbol Connector:TestPoint
- added TP15: VBAT, Relay_THT:Relay_DPDT_Schrack-RT2-FormC_RM5mm, symbol Connector:TestPoint
- added TP16: 0, Relay_THT:Relay_DPDT_Schrack-RT2-FormC_RM5mm, symbol Connector:TestPoint
- added TP17: 1, Relay_THT:Relay_DPDT_Schrack-RT2-FormC_RM5mm, symbol Connector:TestPoint
- added TP18: 2, Relay_THT:Relay_DPDT_Schrack-RT2-FormC_RM5mm, symbol Connector:TestPoint
- added TP19: 3, Relay_THT:Relay_DPDT_Schrack-RT2-FormC_RM5mm, symbol Connector:TestPoint
- added TP20: 4, Relay_THT:Relay_DPDT_Schrack-RT2-FormC_RM5mm, symbol Connector:TestPoint
- added TP21: 5, Relay_THT:Relay_DPDT_Schrack-RT2-FormC_RM5mm, symbol Connector:TestPoint
- added TP22: 6, Relay_THT:Relay_DPDT_Schrack-RT2-FormC_RM5mm, symbol Connector:TestPoint
- added TP23: 7, Relay_THT:Relay_DPDT_Schrack-RT2-FormC_RM5mm, symbol Connector:TestPoint
- added TP24: 8, Relay_THT:Relay_DPDT_Schrack-RT2-FormC_RM5mm, symbol Connector:TestPoint
- added TP25: 9, Relay_THT:Relay_DPDT_Schrack-RT2-FormC_RM5mm, symbol Connector:TestPoint
- added TP26: 10, Relay_THT:Relay_DPDT_Schrack-RT2-FormC_RM5mm, symbol Connector:TestPoint
- added TP27: 11, Relay_THT:Relay_DPDT_Schrack-RT2-FormC_RM5mm, symbol Connector:TestPoint
- C1: value C -> 100nF
- R1: value 2.94 -> 2.94k
- R2: value 2.94 -> 100k
Connections:
- net EN: now also U1.6 (PA5)
- net GND: now also J1.A1 (GND), J1.A12 (GND), J1.B1 (GND), J1.B12 (GND), J1.SH (SHIELD), C6.2, C7.2, C8.2, D1.1 (A1), R6.2, R7.1, SW1.1, SW2.2, TP14.1
- net SCL: now also U1.14 (PB0), R10.2
- net SDA: now also U1.13 (PB1), R11.2
- net STAT: now also U1.8 (PA7)
- net VBAT: now also R10.1, R11.1, TP15.1, TP16.1, TP17.1, TP18.1, TP19.1, TP20.1, TP21.1, TP22.1, TP23.1, TP24.1, TP25.1, TP26.1, TP27.1
- net VBUS: now also J1.A4 (VBUS), J1.A9 (VBUS), J1.B4 (VBUS), J1.B9 (VBUS)
- net VCC: now also C8.1
- net at U1.1 (PA2): now also C7.1, R9.1
- net UDPI: now reaches U1.19 (~{RESET}/PA0)
- net UDPI: now also R12.1, TP12.1
- net at U1.20 (PA1): now also TP13.1
- net at U1.7 (PA6): now also C6.1, R8.1
- net at J1.A5 (CC1): now also R6.1
- net at J1.A7 (D-): now also D1.2 (A2), R12.2
- net at J1.B5 (CC2): now also R7.2
- new net: R9.2, SW2.1
- new net: R8.2, SW1.2
- no-connect marks 0 -> 5
Other:
- moved on the sheet: BT1, C1, C2, C3, C4, C5, IC1, J1, JP1, JP10, JP2, JP3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

Commit message: rearranged
Parts:
- removed BT1: Battery, Package_SON:Texas_DRC0010J_ThermalVias, symbol Device:Battery
- added BAT_GND, BAT_VCC: 5, Relay_THT:Relay_DPDT_Schrack-RT2-FormC_RM5mm, symbol Connector:TestPoint
Connections:
- net GND: now also BAT_GND.1
- net VBAT: now also BAT_VCC.1
- net at IC1.7 (OUT5), TP5.1: now also JP4.1 (A); no longer JP4.2 (B)
- net at IC1.8 (OUT6), TP6.1: now also JP6.2 (B); no longer JP5.1 (A)
- net at IC1.10 (OUT8), JP10.2 (B), TP8.1: now also JP5.1 (A); no longer JP6.2 (B)
- net at IC1.5 (OUT3), JP9.2 (B), TP3.1: now also JP3.2 (B); no longer JP3.1 (A)
- net at IC1.6 (OUT4), TP4.1: now also JP3.1 (A), JP4.2 (B); no longer JP3.2 (B), JP4.1 (A)
Other:
- moved on the sheet: C1, C2, C3, C5, C6, C7, C8, D1, IC1, J1, JP1, JP10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

Commit message: half footprints added
Parts:
- BAT_GND, BAT_VCC, TP12, TP13, TP14, TP15: footprint Relay_THT:Relay_DPDT_Schrack-RT2-FormC_RM5mm -> (none)
- C1: renamed from C8; footprint Package_SO:SOIC-8_3.9x4.9mm_P1.27mm -> Capacitor_SMD:C_0402_1005Metric_Pad0.74x0.62mm_HandSolder
- C2: renamed from C1; footprint Package_SO:SOIC-8_3.9x4.9mm_P1.27mm -> Capacitor_SMD:C_0402_1005Metric_Pad0.74x0.62mm_HandSolder
- C3: renamed from C7; footprint Package_TO_SOT_SMD:SOT-23-5 -> Capacitor_SMD:C_0402_1005Metric_Pad0.74x0.62mm_HandSolder
- C4: renamed from C6; footprint Package_TO_SOT_SMD:SOT-23-5 -> Capacitor_SMD:C_0402_1005Metric_Pad0.74x0.62mm_HandSolder
- C5: renamed from C2; footprint Package_SO:SOIC-8_3.9x4.9mm_P1.27mm -> Capacitor_SMD:C_0402_1005Metric_Pad0.74x0.62mm_HandSolder
- C6: renamed from C3; footprint Package_SO:SOIC-8_3.9x4.9mm_P1.27mm -> (none)
- C7: renamed from C4; footprint Package_TO_SOT_SMD:SOT-23-5 -> (none)
- C8: renamed from C5; footprint Package_TO_SOT_SMD:SOT-23-5 -> (none)
- JP1, JP2, JP6: footprint (none) -> Resistor_SMD:R_0402_1005Metric_Pad0.72x0.64mm_HandSolder
- JP10: renamed from JP7; footprint (none) -> Resistor_SMD:R_0402_1005Metric_Pad0.72x0.64mm_HandSolder
- JP3: renamed from JP9; footprint (none) -> Resistor_SMD:R_0402_1005Metric_Pad0.72x0.64mm_HandSolder
- JP4: renamed from JP3; footprint (none) -> Resistor_SMD:R_0402_1005Metric_Pad0.72x0.64mm_HandSolder
- JP5: renamed from JP4; footprint (none) -> Resistor_SMD:R_0402_1005Metric_Pad0.72x0.64mm_HandSolder
- JP7: renamed from JP5; footprint (none) -> Resistor_SMD:R_0402_1005Metric_Pad0.72x0.64mm_HandSolder
- JP8: renamed from JP10; footprint (none) -> Resistor_SMD:R_0402_1005Metric_Pad0.72x0.64mm_HandSolder
- JP9: renamed from JP8; footprint (none) -> Resistor_SMD:R_0402_1005Metric_Pad0.72x0.64mm_HandSolder
- LED_A0: renamed from TP16; footprint Relay_THT:Relay_DPDT_Schrack-RT2-FormC_RM5mm -> Connector_Wire:SolderWirePad_1x01_SMD_1x2mm
- LED_A1: renamed from TP17; footprint Relay_THT:Relay_DPDT_Schrack-RT2-FormC_RM5mm -> Connector_Wire:SolderWirePad_1x01_SMD_1x2mm
- LED_A10: renamed from TP26; footprint Relay_THT:Relay_DPDT_Schrack-RT2-FormC_RM5mm -> Connector_Wire:SolderWirePad_1x01_SMD_1x2mm
- LED_A11: renamed from TP27; footprint Relay_THT:Relay_DPDT_Schrack-RT2-FormC_RM5mm -> Connector_Wire:SolderWirePad_1x01_SMD_1x2mm
- LED_A2: renamed from TP18; footprint Relay_THT:Relay_DPDT_Schrack-RT2-FormC_RM5mm -> Connector_Wire:SolderWirePad_1x01_SMD_1x2mm
- LED_A3: renamed from TP19; footprint Relay_THT:Relay_DPDT_Schrack-RT2-FormC_RM5mm -> Connector_Wire:SolderWirePad_1x01_SMD_1x2mm
- LED_A4: renamed from TP20; footprint Relay_THT:Relay_DPDT_Schrack-RT2-FormC_RM5mm -> Connector_Wire:SolderWirePad_1x01_SMD_1x2mm
- LED_A5: renamed from TP21; footprint Relay_THT:Relay_DPDT_Schrack-RT2-FormC_RM5mm -> (none)
- LED_A6: renamed from TP22; footprint Relay_THT:Relay_DPDT_Schrack-RT2-FormC_RM5mm -> Connector_Wire:SolderWirePad_1x01_SMD_1x2mm
- LED_A7: renamed from TP23; footprint Relay_THT:Relay_DPDT_Schrack-RT2-FormC_RM5mm -> Connector_Wire:SolderWirePad_1x01_SMD_1x2mm
- LED_A8: renamed from TP24; footprint Relay_THT:Relay_DPDT_Schrack-RT2-FormC_RM5mm -> Connector_Wire:SolderWirePad_1x01_SMD_1x2mm
- LED_A9: renamed from TP25; footprint Relay_THT:Relay_DPDT_Schrack-RT2-FormC_RM5mm -> Connector_Wire:SolderWirePad_1x01_SMD_1x2mm
- LED_K0: renamed from TP0; footprint Relay_THT:Relay_DPDT_Schrack-RT2-FormC_RM5mm -> Connector_Wire:SolderWirePad_1x01_SMD_1x2mm
- LED_K1: renamed from TP1; footprint Relay_THT:Relay_DPDT_Schrack-RT2-FormC_RM5mm -> Connector_Wire:SolderWirePad_1x01_SMD_1x2mm
- LED_K10: renamed from TP10; footprint Relay_THT:Relay_DPDT_Schrack-RT2-FormC_RM5mm -> Connector_Wire:SolderWirePad_1x01_SMD_1x2mm
- LED_K11: renamed from TP11; footprint Relay_THT:Relay_DPDT_Schrack-RT2-FormC_RM5mm -> Connector_Wire:SolderWirePad_1x01_SMD_1x2mm
- LED_K2: renamed from TP2; footprint Relay_THT:Relay_DPDT_Schrack-RT2-FormC_RM5mm -> Connector_Wire:SolderWirePad_1x01_SMD_1x2mm
- LED_K3: renamed from TP3; footprint Relay_THT:Relay_DPDT_Schrack-RT2-FormC_RM5mm -> Connector_Wire:SolderWirePad_1x01_SMD_1x2mm
- LED_K4: renamed from TP4; footprint Relay_THT:Relay_DPDT_Schrack-RT2-FormC_RM5mm -> Connector_Wire:SolderWirePad_1x01_SMD_1x2mm
- LED_K5: renamed from TP5; footprint Relay_THT:Relay_DPDT_Schrack-RT2-FormC_RM5mm -> (none)
- LED_K6: renamed from TP6; footprint Relay_THT:Relay_DPDT_Schrack-RT2-FormC_RM5mm -> Connector_Wire:SolderWirePad_1x01_SMD_1x2mm
- LED_K7: renamed from TP7; footprint Relay_THT:Relay_DPDT_Schrack-RT2-FormC_RM5mm -> Connector_Wire:SolderWirePad_1x01_SMD_1x2mm
- LED_K8: renamed from TP8; footprint Relay_THT:Relay_DPDT_Schrack-RT2-FormC_RM5mm -> Connector_Wire:SolderWirePad_1x01_SMD_1x2mm
- LED_K9: renamed from TP9; footprint Relay_THT:Relay_DPDT_Schrack-RT2-FormC_RM5mm -> Connector_Wire:SolderWirePad_1x01_SMD_1x2mm
- R1, R2: footprint QFN40P300X300X80-21N-D -> Resistor_SMD:R_0402_1005Metric_Pad0.72x0.64mm_HandSolder
- R10, R11, R12, R3, R4, R5, R6, R7, R8, R9: footprint Package_TO_SOT_SMD:SOT-23-5 -> Resistor_SMD:R_0402_1005Metric_Pad0.72x0.64mm_HandSolder
- SW1, SW2: footprint Button_Switch_SMD:Nidec_Copal_CAS-120A -> (none)
Connections:
- no-connect marks 5 -> 15
Other:
- moved on the sheet: C5, C6, IC1, JP1, JP10, JP2, JP3, JP4, JP5, JP6, JP7, JP8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

Commit message: switches updated; basic pcb
Parts:
- removed SW1, SW2: SW_Push, symbol Switch:SW_Push
- added D2: 5V, Diode_SMD:D_SOD-882, symbol Device:D_TVS
- added JP5: (no value), Resistor_SMD:R_0402_1005Metric_Pad0.72x0.64mm_HandSolder, symbol Jumper:Jumper_2_Small_Open
- added S1, S2: EVQ-P7A01P, Library:EVQP7J01P, symbol lib:EVQ-P7A01P
- BAT_GND1: renamed from BAT_GND; footprint (none) -> Connector_Wire:SolderWirePad_1x01_SMD_1x2mm
- BAT_VCC1: renamed from BAT_VCC; value 5 -> 6; footprint (none) -> Connector_Wire:SolderWirePad_1x01_SMD_1x2mm
- C6, C7, C8: footprint (none) -> Capacitor_SMD:C_0603_1608Metric_Pad1.08x0.95mm_HandSolder
- D1: footprint Package_DFN_QFN:QFN-16-1EP_4x4mm_P0.65mm_EP2.1x2.1mm_ThermalVias -> Diode_SMD:D_SOD-882
- IC1: footprint QFN40P300X300X80-21N-D -> Library:QFN40P300X300X80-21N-D
- J1: footprint (none) -> Connector_USB:USB_C_Receptacle_GCT_USB4105-xx-A_16P_TopMnt_Horizontal
- LED_A5, LED_K5, TP12, TP13, TP14, TP15: footprint (none) -> Connector_Wire:SolderWirePad_1x01_SMD_1x2mm
- renumbered JP1 to JP0, JP2 to JP1, JP3 to JP2, JP4 to JP3, JP5 to JP4
Connections:
- net VCC is gone; now on net VBAT: C1.1, C2.2, U1.4 (VCC)
- net GND: now also D2.1 (A1), S1.3 (COM_1), S1.4 (COM_2), S2.3 (COM_1), S2.4 (COM_2)
- net VBUS: now also D2.2 (A2)
- net at IC1.7 (OUT5), JP4.1 (A), LED_K5.1: now also JP5.2 (B)
- net SW1: now reaches C3.1, R9.1, U1.1 (PA2)
- net at R9.2: now also S1.1 (NO_1), S1.2 (NO_2)
- net DBG_TX: now reaches TP13.1, U1.20 (PA1)
- net SW2: now reaches C4.1, R8.1, U1.7 (PA6)
- net at R8.2: now also S2.1 (NO_1), S2.2 (NO_2)
- net at IC1.8 (OUT6), JP6.2 (B), LED_K6.1: now also JP5.1 (A)
- net at D1.2 (A2), J1.A7 (D-), R12.2: now also J1.B7 (D-)
- no-connect marks 15 -> 14
Other:
- moved on the sheet: C3, C4, D1, R1, R2, R8, R9, TP12, TP13, TP14, TP15

Commit message: third of the way there
Connections:
- net EN: now also U1.15 (PC0); no longer U1.6 (PA5)
Other:
- moved on the sheet: R2
Changed lines of the file:
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@@
 	)
 	(junction
-		(at 80.01 139.7)
+		(at 50.8 119.38)
 		(diameter 0)
 		(color 0 0 0 0)
 	)
 	(junction
-		(at 50.8 119.38)
+		(at 30.48 149.86)
 		(diameter 0)
 		(color 0 0 0 0)
@@
 	)
 	(no_connect
-		(at 35.56 149.86)
+		(at 66.04 139.7)
 	)
 	(wire
@@
 	(wire
 		(pts
+			(xy 30.48 149.86) (xy 35.56 149.86)
+		)
+		(stroke
+			(width 0)
+			(type default)
+		)
+	)
+	(wire
+		(pts
 			(xy 229.87 72.39) (xy 229.87 77.47)
 		)
@@
 	(wire
 		(pts
-			(xy 66.04 139.7) (xy 86.36 139.7)
-		)
-		(stroke
-			(width 0)
-			(type default)
-		)
-	)
-	(wire
-		(pts
 			(xy 204.47 57.15) (xy 204.47 77.47)
 		)
@@
 	(wire
 		(pts
+			(xy 30.48 149.86) (xy 30.48 143.51)
+		)
+		(stroke
+			(width 0)
+			(type default)
+		)
+	)
+	(wire
+		(pts
 			(xy 156.21 167.64) (xy 156.21 171.45)
 		)
@@
 	)
 	(label "EN"
-		(at 86.36 139.7 180)
+		(at 30.48 143.51 270)
 		(effects
 			(font
@@
 	(symbol
 		(lib_id "Device:R")
-		(at 80.01 135.89 180)
+		(at 26.67 149.86 270)
 		(unit 1)
 		(body_style 1)
@@
 		(dnp no)
 		(property "Reference" "R2"
-			(at 82.804 134.366 90)
+			(at 25.146 147.066 90)
 			(show_name no)
 			(do_not_autoplace no)
@@
 		)
 		(property "Value" "100k"
-			(at 77.724 133.604 90)
+			(at 24.384 152.146 90)
 			(show_name no)
 			(do_not_autoplace no)
@@
 		)
 		(property "Footprint" "Resistor_SMD:R_0402_1005Metric_Pad0.72x0.64mm_HandSolder"
-			(at 81.788 135.89 90)
+			(at 26.67 148.082 90)
 			(hide yes)
 			(show_name no)
@@
 		)
 		(property "Datasheet" ""
-			(at 80.01 135.89 0)
+			(at 26.67 149.86 0)
 			(hide yes)
 			(show_name no)
@@
 		)
 		(property "Description" "Resistor"
-			(at 80.01 135.89 0)
+			(at 26.67 149.86 0)
 			(hide yes)
 			(show_name no)
@@
 	(symbol
 		(lib_id "power:GND")
-		(at 80.01 132.08 180)
+		(at 22.86 149.86 270)
 		(unit 1)
 		(body_style 1)
@@
 		(dnp no)
 		(property "Reference" "#PWR011"
-			(at 80.01 125.73 0)
+			(at 16.51 149.86 0)
 			(hide yes)
 			(show_name no)
@@
 		)
 		(property "Value" "GND"
-			(at 77.216 130.556 90)
+			(at 21.336 152.654 90)
 			(show_name no)
 			(do_not_autoplace no)
@@
 		)
 		(property "Footprint" ""
-			(at 80.01 132.08 0)
+			(at 22.86 149.86 0)
 			(hide yes)
 			(show_name no)
@@
 		)
 		(property "Datasheet" ""
-			(at 80.01 132.08 0)
+			(at 22.86 149.86 0)
 			(hide yes)
 			(show_name no)
@@
 		)
 		(property "Description" "Power symbol creates a global label with name \"GND\" , ground"
-			(at 80.01 132.08 0)
+			(at 22.86 149.86 0)
 			(hide yes)
 			(show_name no)

Commit message: foottoprinto
Connections:
- net EN: now also U1.11 (PB3); no longer U1.15 (PC0)
- net STAT: now also U1.6 (PA5); no longer U1.8 (PA7)
- net SW1: now also U1.7 (PA6); no longer U1.1 (PA2)
- net SW2: now also U1.8 (PA7); no longer U1.7 (PA6)
Other:
- moved on the sheet: R2
Changed lines of the file:
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@@
 	)
 	(junction
-		(at 30.48 149.86)
+		(at 48.26 76.2)
 		(diameter 0)
 		(color 0 0 0 0)
 	)
 	(junction
-		(at 48.26 76.2)
+		(at 194.31 77.47)
 		(diameter 0)
 		(color 0 0 0 0)
 	)
 	(junction
-		(at 194.31 77.47)
+		(at 85.09 160.02)
 		(diameter 0)
 		(color 0 0 0 0)
 	)
 	(junction
-		(at 85.09 160.02)
+		(at 69.85 167.64)
 		(diameter 0)
 		(color 0 0 0 0)
@@
 	)
 	(no_connect
-		(at 66.04 157.48)
-	)
-	(no_connect
 		(at 63.5 55.88)
 	)
@@
 	)
 	(no_connect
-		(at 35.56 154.94)
+		(at 35.56 149.86)
 	)
 	(no_connect
-		(at 66.04 139.7)
+		(at 66.04 132.08)
+	)
+	(no_connect
+		(at 35.56 154.94)
 	)
 	(wire
@@
 	(wire
 		(pts
+			(xy 66.04 157.48) (xy 69.85 157.48)
+		)
+		(stroke
+			(width 0)
+			(type default)
+		)
+	)
+	(wire
+		(pts
 			(xy 214.63 17.78) (xy 214.63 21.59)
 		)
@@
 	(wire
 		(pts
-			(xy 30.48 149.86) (xy 35.56 149.86)
-		)
-		(stroke
-			(width 0)
-			(type default)
-		)
-	)
-	(wire
-		(pts
 			(xy 229.87 72.39) (xy 229.87 77.47)
 		)
@@
 	(wire
 		(pts
-			(xy 30.48 149.86) (xy 30.48 143.51)
+			(xy 69.85 157.48) (xy 69.85 167.64)
+		)
+		(stroke
+			(width 0)
+			(type default)
+		)
+	)
+	(wire
+		(pts
+			(xy 69.85 167.64) (xy 63.5 167.64)
 		)
 		(stroke
@@
 	)
 	(label "SW2"
-		(at 66.04 142.24 0)
+		(at 66.04 144.78 0)
 		(effects
 			(font
@@
 	)
 	(label "STAT"
-		(at 66.04 144.78 0)
+		(at 66.04 139.7 0)
 		(effects
 			(font
@@
 	)
 	(label "EN"
-		(at 30.48 143.51 270)
+		(at 63.5 167.64 0)
 		(effects
 			(font
 				(size 1.27 1.27)
 			)
-			(justify right bottom)
+			(justify left bottom)
 		)
 	)
 	(label "SW1"
-		(at 66.04 132.08 0)
+		(at 66.04 142.24 0)
 		(effects
 			(font
@@
 	(symbol
 		(lib_id "Device:R")
-		(at 26.67 149.86 270)
+		(at 69.85 171.45 0)
 		(unit 1)
 		(body_style 1)
@@
 		(dnp no)
 		(property "Reference" "R2"
-			(at 25.146 147.066 90)
+			(at 67.056 172.974 90)
 			(show_name no)
 			(do_not_autoplace no)
@@
 		)
 		(property "Value" "100k"
-			(at 24.384 152.146 90)
+			(at 72.136 173.736 90)
 			(show_name no)
 			(do_not_autoplace no)
@@
 		)
 		(property "Footprint" "Resistor_SMD:R_0402_1005Metric_Pad0.72x0.64mm_HandSolder"
-			(at 26.67 148.082 90)
+			(at 68.072 171.45 90)
 			(hide yes)
 			(show_name no)
@@
 		)
 		(property "Datasheet" ""
-			(at 26.67 149.86 0)
+			(at 69.85 171.45 0)
 			(hide yes)
 			(show_name no)
@@
 		)
 		(property "Description" "Resistor"
-			(at 26.67 149.86 0)
+			(at 69.85 171.45 0)
 			(hide yes)
 			(show_name no)
@@
 	(symbol
 		(lib_id "power:GND")
-		(at 22.86 149.86 270)
+		(at 69.85 175.26 0)
 		(unit 1)
 		(body_style 1)
@@
 		(dnp no)
 		(property "Reference" "#PWR011"
-			(at 16.51 149.86 0)
+			(at 69.85 181.61 0)
 			(hide yes)
 			(show_name no)
@@
 		)
 		(property "Value" "GND"
-			(at 21.336 152.654 90)
+			(at 72.644 176.784 90)
 			(show_name no)
 			(do_not_autoplace no)
@@
 		)
 		(property "Footprint" ""
-			(at 22.86 149.86 0)
+			(at 69.85 175.26 0)
 			(hide yes)
 			(show_name no)
@@
 		)
 		(property "Datasheet" ""
-			(at 22.86 149.86 0)
+			(at 69.85 175.26 0)
 			(hide yes)
 			(show_name no)
@@
 		)
 		(property "Description" "Power symbol creates a global label with name \"GND\" , ground"
-			(at 22.86 149.86 0)
+			(at 69.85 175.26 0)
 			(hide yes)
 			(show_name no)

Commit message: output; SAD_grbr; SAD_bom
Parts:
- BAT_GND1, BAT_VCC1, JP0, JP1, JP10, JP2, JP3, JP4, JP5, JP6, JP7, JP8, JP9, TP12, TP13, TP14, TP15: Manufacturer_Name (none) -> -; Manufacturer_Part_Number (none) -> -; now left out of the parts list
- C1, C5: Manufacturer_Name (none) -> Samsung; Manufacturer_Part_Number (none) -> CL05A105KP5NNNC
- C2: Manufacturer_Name (none) -> Murata; Manufacturer_Part_Number (none) -> GRM155R71C104KA88D
- C3, C4: Manufacturer_Name (none) -> Murata; Manufacturer_Part_Number (none) -> GRM155R71H103KA88D
- C6, C7, C8: Manufacturer_Name (none) -> Samsung; Manufacturer_Part_Number (none) -> CL10A475KO8NNNC
- D1, D2: Manufacturer_Name (none) -> Texas Instruments; Manufacturer_Part_Number (none) -> TPD1E10B06DPYR
- J1: Manufacturer_Name (none) -> GCT; Manufacturer_Part_Number (none) -> USB4105-GF-A
- LED_A0, LED_K0: value 0 -> (none); Manufacturer_Name (none) -> -; Manufacturer_Part_Number (none) -> -; now left out of the parts list
- LED_A1, LED_K1: value 1 -> (none); Manufacturer_Name (none) -> -; Manufacturer_Part_Number (none) -> -; now left out of the parts list
- LED_A10, LED_K10: value 10 -> (none); Manufacturer_Name (none) -> -; Manufacturer_Part_Number (none) -> -; now left out of the parts list
- LED_A11, LED_K11: value 11 -> (none); Manufacturer_Name (none) -> -; Manufacturer_Part_Number (none) -> -; now left out of the parts list
- LED_A2, LED_K2: value 2 -> (none); Manufacturer_Name (none) -> -; Manufacturer_Part_Number (none) -> -; now left out of the parts list
- LED_A3, LED_K3: value 3 -> (none); Manufacturer_Name (none) -> -; Manufacturer_Part_Number (none) -> -; now left out of the parts list
- LED_A4, LED_K4: value 4 -> (none); Manufacturer_Name (none) -> -; Manufacturer_Part_Number (none) -> -; now left out of the parts list
- LED_A5, LED_K5: value 5 -> (none); Manufacturer_Name (none) -> -; Manufacturer_Part_Number (none) -> -; now left out of the parts list
- LED_A6, LED_K6: value 6 -> (none); Manufacturer_Name (none) -> -; Manufacturer_Part_Number (none) -> -; now left out of the parts list
- LED_A7, LED_K7: value 7 -> (none); Manufacturer_Name (none) -> -; Manufacturer_Part_Number (none) -> -; now left out of the parts list
- LED_A8, LED_K8: value 8 -> (none); Manufacturer_Name (none) -> -; Manufacturer_Part_Number (none) -> -; now left out of the parts list
- LED_A9, LED_K9: value 9 -> (none); Manufacturer_Name (none) -> -; Manufacturer_Part_Number (none) -> -; now left out of the parts list
- R1: Manufacturer_Name (none) -> YAGEO; Manufacturer_Part_Number (none) -> RC0402FR-072K94L
- R10, R11, R4: Manufacturer_Name (none) -> YAGEO; Manufacturer_Part_Number (none) -> RC0402FR-074K7L
- R12, R8, R9: Manufacturer_Name (none) -> YAGEO; Manufacturer_Part_Number (none) -> RC0402FR-071KL
- R2: Manufacturer_Name (none) -> YAGEO; Manufacturer_Part_Number (none) -> RC0402FR-07100KL
- R3: Manufacturer_Name (none) -> YAGEO; Manufacturer_Part_Number (none) -> RC0402FR-076K8L
- R5: Manufacturer_Name (none) -> YAGEO; Manufacturer_Part_Number (none) -> RC0402FR-071ML
- R6, R7: Manufacturer_Name (none) -> YAGEO; Manufacturer_Part_Number (none) -> RC0402FR-075K1L
- U1: Manufacturer_Name (none) -> Microchip; Manufacturer_Part_Number (none) -> ATTINY1616-MNR
- U2: Manufacturer_Name (none) -> Microchip; Manufacturer_Part_Number (none) -> MCP73831T-2ACI/OT
